File: hackpad/PCB/hackpad.kicad_pcb (KiCad board)
At the start: 2 copper layers, 69.1 x 90.5 mm, 7 parts, among them SW1 SW_Push, SW2 SW_Push, SW3 SW_Push, SW4 SW_Push, U1 XIAO-RP2040-DIP

Commit message: Add files via upload
Parts:
- D1, D2: value SK6812MINI -> SK6812MINI E; footprint LED_SMD:LED_SK6812MINI_PLCC4_3.5x3.5mm_P1.75mm -> Library:LED_SK6812-E
- turned D1 to 180 degrees
- turned D2 to 180 degrees
Routing:
- net GND: track 174.7 -> 111.9 mm
- net +5V: track 77.9 -> 93.2 mm
- net Net-(D1-DOUT): track 15.8 -> 21.4 mm
