File: hackpad/PCB/hackpad.kicad_sch (KiCad schematic)
At the start: 7 parts, among them SW1 SW_Push, SW2 SW_Push, SW3 SW_Push, SW4 SW_Push, U1 XIAO-RP2040-DIP

Commit message: Add files via upload
Parts:
- D1, D2: value SK6812MINI -> SK6812MINI E; footprint LED_SMD:LED_SK6812MINI_PLCC4_3.5x3.5mm_P1.75mm -> Library:LED_SK6812-E
Connections:
- no-connect marks 0 -> 1
Changed lines of the file:
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@@
 		(color 0 0 0 0)
+	)
+	(no_connect
+		(at 113.03 137.16)
 	)
 	(wire
@@
 			)
 		)
-		(property "Value" "SK6812MINI"
+		(property "Value" "SK6812MINI E"
 			(at 118.11 133.2798 0)
 			(effects
@@
 			)
 		)
-		(property "Footprint" "LED_SMD:LED_SK6812MINI_PLCC4_3.5x3.5mm_P1.75mm"
+		(property "Footprint" "Library:LED_SK6812-E"
 			(at 106.68 144.78 0)
 			(effects
@@
 			)
 		)
-		(property "Value" "SK6812MINI"
+		(property "Value" "SK6812MINI E"
 			(at 91.44 133.2798 0)
 			(effects
@@
 			)
 		)
-		(property "Footprint" "LED_SMD:LED_SK6812MINI_PLCC4_3.5x3.5mm_P1.75mm"
+		(property "Footprint" "Library:LED_SK6812-E"
 			(at 80.01 144.78 0)
 			(effects
